Commit message: update 17/01

File: ros-bioloid/src/bioloid_master/urdf/mioloid_robot_head.urdf (robot description, URDF)
Before this commit: robot bioloid, 27 links, 26 joints
Joints:
- joint left_hip_swing_joint: limit lower=-1.570795 upper=1.9 effort=10 velocity=1.0 -> lower=-0.5 upper=2 effort=10 velocity=1.0
- joint right_hip_swing_joint: limit lower=-1.570795 upper=1.9 effort=10 velocity=1.0 -> lower=-0.5 upper=2 effort=10 velocity=1.0
- joint right_knee_joint: limit lower=-2.4 upper=0.0 effort=10 velocity=1.0 -> lower=-2.3 upper=0.0 effort=10 velocity=1.0
